File: eagle/untitled.sch (EAGLE design)
At the start: 30 parts, among them IC1 74HC595D, IC2 74HC595D, Q1 BC557, Q2 BC557, Q3 BC557, Q4 BC557, Q5 BC557, Q6 BC547, Q7 BC547, Q8 BC547

Commit message: Исправления схемы.
Parts:
- added R12, R13, R14, R15: 4.7K, rcl:R-EU_M0805
- added R16, R17: 300, rcl:R-EU_M0805
- added U2: DC-DC-STEP-UP-MT3608, diy-modules:DC-DC-STEP-UP-MT3608
- renumbered U$1 to U1
Connections:
- new net N$25: Q4.B, R16.2
- new net N$26: Q5.B, R17.2
- net +24V: now also U2.OUT+
- net A11: now also R12.1
- net A13: now also R13.1
- net A15: now also R14.1
- net GND: now also R12.2, R13.2, R14.2, R15.2, U1.GND2, U2.IN-, U2.OUT-
- net N$10: now also R16.1; no longer Q4.B
- net N$12: now also R17.1; no longer Q5.B
- net N$19: now also Q7.C; no longer Q6.C
- net N$21: now also Q7.B; no longer Q6.B
- net N$22: now also Q6.C; no longer Q7.C
- net N$24: now also Q6.B; no longer Q7.B
- net OE: now also R15.1
- net VCC: now also U2.IN+
Other:
- moved on the sheet: D5, J1, Q4, Q5, Q6, Q7, X1-1, X1-2
